Commit message: Prepare Avance 3 physical integration safely

File: src/thesis_simulation/urdf/jaco_gazebo.ros2_control.xacro (robot description, xacro)
@@ -3,4 +3,20 @@
     xmlns:xacro="http://www.ros.org/wiki/xacro"
     name="j2n6s300_gazebo">
+  <xacro:arg name="initial_pose" default="default"/>
+  <xacro:property
+      name="use_z_ready"
+      value="${'$(arg initial_pose)' == 'z_ready'}"/>
+  <xacro:property name="joint_1_initial" value="0.0"/>
+  <xacro:property
+      name="joint_2_initial"
+      value="${2.6179938779914944 if use_z_ready else 3.141592653589793}"/>
+  <xacro:property
+      name="joint_3_initial"
+      value="${3.6651914291880923 if use_z_ready else 3.141592653589793}"/>
+  <xacro:property name="joint_4_initial" value="0.0"/>
+  <xacro:property
+      name="joint_5_initial"
+      value="${0.3490658503988659 if use_z_ready else 0.0}"/>
+  <xacro:property name="joint_6_initial" value="0.0"/>
   <!-- =========================================================
        Common JACO geometry and kinematics
@@ -32,5 +48,5 @@
       <command_interface name="position"/>
       <state_interface name="position">
-        <param name="initial_value">0.0</param>
+        <param name="initial_value">${joint_1_initial}</param>
       </state_interface>
       <state_interface name="velocity"/>
@@ -39,5 +55,5 @@
       <command_interface name="position"/>
       <state_interface name="position">
-        <param name="initial_value">3.141592653589793</param>
+        <param name="initial_value">${joint_2_initial}</param>
       </state_interface>
       <state_interface name="velocity"/>
@@ -46,5 +62,5 @@
       <command_interface name="position"/>
       <state_interface name="position">
-        <param name="initial_value">3.141592653589793</param>
+        <param name="initial_value">${joint_3_initial}</param>
       </state_interface>
       <state_interface name="velocity"/>
@@ -53,5 +69,5 @@
       <command_interface name="position"/>
       <state_interface name="position">
-        <param name="initial_value">0.0</param>
+        <param name="initial_value">${joint_4_initial}</param>
       </state_interface>
       <state_interface name="velocity"/>
@@ -60,5 +76,5 @@
       <command_interface name="position"/>
       <state_interface name="position">
-        <param name="initial_value">0.0</param>
+        <param name="initial_value">${joint_5_initial}</param>
       </state_interface>
       <state_interface name="velocity"/>
@@ -67,5 +83,5 @@
       <command_interface name="position"/>
       <state_interface name="position">
-        <param name="initial_value">0.0</param>
+        <param name="initial_value">${joint_6_initial}</param>
       </state_interface>
       <state_interface name="velocity"/>
